File: Electrical_Slip_Ring.kicad_pcb (KiCad board)
At the start: 2 copper layers, 0 parts

Commit message: Create edge of rotor.
Other:
- board outline added: 93 x 93 mm
- copper layers 2 -> 4
Changed lines of the file:
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@@
 (kicad_pcb (version 20211014) (generator pcbnew)
   (general
-    (thickness 1.6)
+    (thickness 1.59)
   )
   (paper "A4")
   (layers
     (0 "F.Cu" signal)
+    (1 "In1.Cu" signal)
+    (2 "In2.Cu" signal)
     (31 "B.Cu" signal)
     (32 "B.Adhes" user "B.Adhesive")
@@
     (48 "B.Fab" user)
     (49 "F.Fab" user)
-    (50 "User.1" user)
-    (51 "User.2" user)
-    (52 "User.3" user)
-    (53 "User.4" user)
-    (54 "User.5" user)
-    (55 "User.6" user)
-    (56 "User.7" user)
-    (57 "User.8" user)
-    (58 "User.9" user)
   )
   (setup
+    (stackup
+      (layer "F.SilkS" (type "Top Silk Screen") (color "White"))
+      (layer "F.Paste" (type "Top Solder Paste"))
+      (layer "F.Mask" (type "Top Solder Mask") (color "Green") (thickness 0.01))
+      (layer "F.Cu" (type "copper") (thickness 0.035))
+      (layer "dielectric 1" (type "prepreg") (thickness 0.2) (material "PP") (epsilon_r 4.6) (loss_tangent 0.02))
+      (layer "In1.Cu" (type "copper") (thickness 0.0175))
+      (layer "dielectric 2" (type "core") (thickness 1.065) (material "FR4") (epsilon_r 4.5) (loss_tangent 0.02))
+      (layer "In2.Cu" (type "copper") (thickness 0.0175))
+      (layer "dielectric 3" (type "prepreg") (thickness 0.2) (material "PP") (epsilon_r 4.6) (loss_tangent 0.02))
+      (layer "B.Cu" (type "copper") (thickness 0.035))
+      (layer "B.Mask" (type "Bottom Solder Mask") (color "Green") (thickness 0.01))
+      (layer "B.Paste" (type "Bottom Solder Paste"))
+      (layer "B.SilkS" (type "Bottom Silk Screen") (color "White"))
+      (copper_finish "None")
+      (dielectric_constraints no)
+    )
     (pad_to_mask_clearance 0)
     (pcbplotparams
@@
   )
   (net 0 "")
+  (gr_circle (center 100 100) (end 143.5 100) (layer "F.Cu") (width 1.5) (fill none))
+  (gr_circle (center 100 100) (end 139.5 100) (layer "F.Cu") (width 1.5) (fill none))
+  (gr_circle (center 100 100) (end 141.5 100) (layer "F.Cu") (width 1) (fill none))
+  (gr_circle (center 100 100) (end 139.5 100) (layer "B.Cu") (width 1.5) (fill none))
+  (gr_circle (center 100 100) (end 143.5 100) (layer "B.Cu") (width 1.5) (fill none))
+  (gr_circle (center 100 100) (end 141.5 100) (layer "B.Cu") (width 1) (fill none))
+  (gr_circle (center 100 100) (end 139.5 100) (layer "B.Mask") (width 1.5) (fill none))
+  (gr_circle (center 100 100) (end 143.5 100) (layer "B.Mask") (width 1.5) (fill none))
+  (gr_circle (center 100 100) (end 141.5 100) (layer "B.Mask") (width 1) (fill none))
+  (gr_circle (center 100 100) (end 139.5 100) (layer "F.Mask") (width 1.5) (fill none))
+  (gr_circle (center 100 100) (end 141.5 100) (layer "F.Mask") (width 1) (fill none))
+  (gr_circle (center 100 100) (end 143.5 100) (layer "F.Mask") (width 1.5) (fill none))
   (gr_circle (center 100 100) (end 135 100) (layer "Dwgs.User") (width 0.1) (fill none))
   (gr_circle (center 100 100) (end 150 100) (layer "Dwgs.User") (width 0.1) (fill none))
+  (gr_line (start 139.5 100) (end 143.5 100) (layer "Dwgs.User") (width 0.15))
+  (gr_line (start 139.5 99.5) (end 139.5 100.5) (layer "Dwgs.User") (width 0.15))
   (gr_rect (start 135 95) (end 136 105) (layer "Dwgs.User") (width 0.1) (fill none))
   (gr_circle (center 100 100) (end 148.5 100) (layer "Dwgs.User") (width 0.1) (fill none))
   (gr_rect (start 147 95) (end 148 105) (layer "Dwgs.User") (width 0.1) (fill none))
   (gr_circle (center 100 100) (end 133.5 100) (layer "Dwgs.User") (width 0.1) (fill none))
+  (gr_line (start 143.5 99.5) (end 143.5 100.5) (layer "Dwgs.User") (width 0.15))
+  (gr_line (start 95 136.25) (end 94.997389 134.893214) (layer "Edge.Cuts") (width 0.1))
+  (gr_line (start 94.75 136.624999) (end 95 136.25) (layer "Edge.Cuts") (width 0.1))
+  (gr_line (start 99.75 63) (end 100 63.25) (layer "Edge.Cuts") (width 0.1))
+  (gr_arc (start 100 135.25) (mid 97.492341 135.16069) (end 94.997389 134.893214) (layer "Edge.Cuts") (width 0.1))
+  (gr_line (start 136.625 105.25) (end 136.25 105) (layer "Edge.Cuts") (width 0.1))
+  (gr_line (start 63.375001 94.75) (end 63.75 95) (layer "Edge.Cuts") (width 0.1))
+  (gr_arc (start 136.624999 105.25) (mid 124.32968 127.875073) (end 100.24999 136.998521) (layer "Edge.Cuts") (width 0.1))
+  (gr_arc (start 135.25 100) (mid 135.16069 102.507659) (end 134.893214 105.002611) (layer "Edge.Cuts") (width 0.1))
+  (gr_line (start 100.25 137) (end 100 136.75) (layer "Edge.Cuts") (width 0.1))
+  (gr_line (start 105 63.75) (end 105.002611 65.106786) (layer "Edge.Cuts") (width 0.1))
+  (gr_line (start 105.25 63.375001) (end 105 63.75) (layer "Edge.Cuts") (width 0.1))
+  (gr_arc (start 94.75 136.624998) (mid 72.124928 124.32968) (end 63.00148 100.24999) (layer "Edge.Cuts") (width 0.1))
+  (gr_line (start 63.75 95) (end 65.106786 94.997389) (layer "Edge.Cuts") (width 0.1))
+  (gr_line (start 63.25 100) (end 64.75 100) (layer "Edge.Cuts") (width 0.1))
+  (gr_arc (start 63.375002 94.75) (mid 75.67032 72.124928) (end 99.75001 63.00148) (layer "Edge.Cuts") (width 0.1))
+  (gr_line (start 136.25 105) (end 134.893214 105.002611) (layer "Edge.Cuts") (width 0.1))
+  (gr_circle (center 100 100) (end 146.5 100) (layer "Edge.Cuts") (width 0.1) (fill none))
+  (gr_arc (start 64.75 100) (mid 64.83931 97.492341) (end 65.106786 94.997389) (layer "Edge.Cuts") (width 0.1))
+  (gr_line (start 100 63.25) (end 100 64.75) (layer "Edge.Cuts") (width 0.1))
+  (gr_line (start 137 99.75) (end 136.75 100) (layer "Edge.Cuts") (width 0.1))
+  (gr_line (start 136.75 100) (end 135.25 100) (layer "Edge.Cuts") (width 0.1))
+  (gr_arc (start 100 64.75) (mid 102.507659 64.83931) (end 105.002611 65.106786) (layer "Edge.Cuts") (width 0.1))
+  (gr_arc (start 105.25 63.375002) (mid 127.875072 75.67032) (end 136.99852 99.75001) (layer "Edge.Cuts") (width 0.1))
+  (gr_line (start 63 100.25) (end 63.25 100) (layer "Edge.Cuts") (width 0.1))
+  (gr_line (start 100 136.75) (end 100 135.25) (layer "Edge.Cuts") (width 0.1))
   (gr_circle (center 100 100) (end 146.5 100) (layer "F.Fab") (width 0.1) (fill none))
+  (gr_line (start 134.893214 105.002611) (end 136.25 105) (layer "F.Fab") (width 0.1))
+  (gr_line (start 136.75 100) (end 135.25 100) (layer "F.Fab") (width 0.1))
+  (gr_arc (start 135.25 100) (mid 135.16069 102.507659) (end 134.893214 105.002611) (layer "F.Fab") (width 0.1))
   (gr_circle (center 100 100) (end 137 100) (layer "F.Fab") (width 0.1) (fill none))
-  (gr_rect (start 137.65 94.5) (end 145.35 105.5) (layer "F.Fab") (width 0.1) (fill none))
+  (gr_line (start 137 99.75) (end 136.75 100) (layer "F.Fab") (width 0.1))
+  (gr_line (start 136.25 105) (end 136.625 105.25) (layer "F.Fab") (width 0.1))
   (target plus (at 100 100) (size 5) (width 0.1) (layer "Edge.Cuts"))
 )
