File: OUTER_HOLDER/OUTER_HOLDER.kicad_pcb (KiCad board)
At the start: 2 copper layers, 10 x 45 mm, 1 part

Commit message: Update OUTER_HOLDER.kicad_pcb
Routing:
- net (no net): track 305.5 -> 329.2 mm
